Commit message: Integrate simple hand

File: r2p_description/urdf/r2p.xacro (robot description, xacro)
@@ -8,4 +8,5 @@
   <xacro:include filename="$(find r2p_sea_arm_description)/urdf/r2p_sea_arm_right.xacro" />
   <!-- Link both arms on a tripod -->
+  <xacro:include filename="$(find r2p_simple_hand_description)/urdf/r2p_simple_hand_right.xacro" />
   <!-- Tripod Link -->
   <link name="tripod_link">
@@ -66,4 +67,10 @@
     <origin xyz="-0.0165 -0.09 0.9" rpy="0 0 ${22*pi/180}"/>
   </joint>
+  <!-- Fix the simple hand to the arm -->
+  <joint name="right_elbow_simple_hand_hook_fixed" type="fixed">
+    <parent link="right_elbow_link"/>
+    <child link="right_simple_hand_hook_link"/>
+    <origin xyz="0 0 0" rpy="0 0 0"/>
+  </joint>
   <!-- Fix the tripod on the base -->
   <joint name="base_tripod_fixed" type="fixed">

Commit message: New branch and new tripod model values

File: r2p_description/urdf/r2p.xacro (robot description, xacro)
@@ -14,5 +14,5 @@
       <origin xyz="0 0 0" rpy="0 0 0"/>
       <geometry>
-	    <mesh filename="package://r2p_description/meshes/visual/tripod_link.dae"/>
+	    <mesh filename="package://r2p_description/meshes/visual/tripod_link_80.dae"/>
       </geometry>
     </visual>
@@ -20,5 +20,5 @@
       <origin xyz="0 0 0" rpy="0 0 0"/>
       <geometry>
-	    <mesh filename="package://r2p_description/meshes/collision/tripod_link_collision.stl"/>
+	    <mesh filename="package://r2p_description/meshes/collision/tripod_link_80_collision.stl"/>
       </geometry>
     </collision>
@@ -65,5 +65,5 @@
     <parent link="tripod_link"/>
     <child link="right_arm_link"/>
-    <origin xyz="-0.0165 -0.09 0.9" rpy="0 0 ${22*pi/180}"/>
+    <origin xyz="-0.0165 -0.09 0.8" rpy="0 0 ${22*pi/180}"/>
   </joint>
   <!-- Fix the simple hand to the arm -->
@@ -77,5 +77,5 @@
     <parent link="base_link"/>
     <child link="tripod_link"/>
-    <origin xyz="0 0 0.13" rpy="0 0 0"/>
+    <origin xyz="0 0 0.15" rpy="0 0 0"/>
   </joint>
 </robot>
